Commit message: adjusting model and stls to work with gripper

File: src/db_support/urdf/dodobot.urdf (robot description, URDF)
Before this commit: robot dodobot, 2 links, 1 joints
Links:
- added link camera_rotate_link; visual mesh filename=package://db_support/meshes/camera.stl
- added link linear_base_link
- added link linear_link; visual mesh filename=package://db_support/meshes/gripper.stl
- link tilt_base_link: geometry 
Joints:
- removed joint base_link_to_camera_joint
- added joint base_link_to_tilt_base_joint: type fixed, parent base_link, child tilt_base_link, origin xyz=0.04796 0.0 0.24785
- added joint linear_base_to_base_link: type fixed, parent base_link, child linear_base_link, origin xyz=0.06046488 0.0 0.01825032
- added joint linear_to_linear_base_link: type prismatic, parent linear_base_link, child linear_link, origin xyz=0 0 0, axis 0 0 1, limit lower=0 upper=0.154 effort=1000.0 velocity=0.5
- added joint tilt_base_to_camera_rotate_joint: type revolute, parent tilt_base_link, child camera_rotate_link, origin xyz=0 0 0, axis 0 1 0, limit lower=0.0 upper=0.548 effort=1000.0 velocity=0.5

Commit message: adding joint state publisher. tweaking rtabmap parameters

File: src/db_support/urdf/dodobot.urdf (robot description, URDF)
Before this commit: robot dodobot, 5 links, 4 joints
Links:
- removed link base_link
- added link wheel_center_link; visual mesh filename=package://db_support/meshes/chassis.stl
Joints:
- joint base_link_to_tilt_base_joint: parent base_link -> wheel_center_link
- joint linear_base_to_base_link: parent base_link -> wheel_center_link
